File: docs/img/aux/aux.kicad_sch (KiCad schematic)
At the start: 2 parts

Commit message: mas
Parts:
- added BZ? (x2): Buzzer, symbol Device:Buzzer
- added Q?: Q_NPN_BCE, symbol Device:Q_NPN_BCE
- added Q?: Q_PNP_BCE, symbol Device:Q_PNP_BCE
- added R? (x2): 1k, symbol Device:R
Connections:
- new net: Q?.1 (B), R?.2 (x2)
- new net: BZ?.2 (+), Q?.2 (C)
- new net: BZ?.1 (-), Q?.2 (C)
- new net +5V: BZ?.1 (-), Q?.3 (E)
- new net Earth: BZ?.2 (+), Q?.3 (E)
- new net GPIO: R?.1, R?.1
